Commit message: Update and rename ros.u to ros.xacro

File: ros.xacro (robot description, xacro)
@@ -55,53 +55,2 @@
 </joint>
 </robot>
-<!-- <?xml version="1.0"?>
-<robot name="my_robot">
-    <link name="base_footprint"/>
-    <link name="chassis">
-        <visual>
-            <origin rpy="0 0 0" xyz="0 0 0" />
-            <geometry>
-                <box size="0.1 0.1 0.05" />
-            </geometry>
-            <material>
-                <color rgba="1.0 1 1.0 1.0"/>
-            </material>
-        </visual>
-        <collision>
-            <origin rpy="0 0 0" xyz="0 0 0" />
-            <geometry>
-                <box size="0.1 0.1 0.05" />
-            </geometry>
-        </collision>
-    </link>
-    <joint name="chassis_base_footprint" type="fixed">
-        <origin xyz="0.0 0.0 0.0" rpy="0.0 0.0 0.0"/>
-        <parent link="base_footprint"/>
-        <child link="chassis"/>
-        <axis xyz="0.0 0.0 0.0"/>
-    </joint>
-  <!-- Link: Hemisphere -->
-    <link name="lidar">
-        <visual>
-            <origin rpy="0 0 0" xyz="0 0 0" />
-            <geometry>
-                <sphere radius="0.025" />
-            </geometry>
-            <material>
-                <color rgba="0.0 0.0 1.0 1.0"/>
-            </material>
-        </visual>
-        <collision>
-            <origin rpy="0 0 0" xyz="0 0 0" />
-            <geometry>
-                <box size="0.1 0.1 0.05" />
-            </geometry>
-        </collision>
-    </link>
-  <!-- Joint: Fixed (connects Rectangle and Hemisphere) -->
-    <joint name="base_lidar" type="fixed">
-        <origin rpy="0 0 0" xyz="0 0 0.025" />
-        <parent link="base_footprint" />
-        <child link="lidar" />
-    </joint>
-</robot> -->
